File: TSOC_RS485_EM/TSOC_RS485_EM.sch (EAGLE design)
At the start: 41 parts, among them Q1 FDC6420C, Q2 MOSFET-NCHANNELAO3404A, U1 ST1480ACSOIC, U2 ATMEGA328, U3 MIC5219 3.3V, U4 NCP361SNT1G, X1 RESONATORSMD

Commit message: update user docs
Other:
- note added: "thingSoC Reference Design Open Source Sockets for IoT"
Changed lines of the file:
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@@
 (or Expansion)
 Board Selection</text>
-<text x="363.22" y="383.54" size="2.54" layer="91" font="vector" ratio="15" rot="R180">ThingSoC Base
-(or Expansion)
-Board Selection</text>
+<text x="195.58" y="25.4" size="2.54" layer="91" font="vector" ratio="15">thingSoC Reference Design
+Open Source Sockets for IoT</text>
+<text x="195.58" y="243.84" size="2.54" layer="91" font="vector" ratio="15">thingSoC Reference Design
+Open Source Sockets for IoT</text>
+<text x="477.52" y="243.84" size="2.54" layer="91" font="vector" ratio="15">thingSoC Reference Design
+Open Source Sockets for IoT</text>
+<text x="477.52" y="25.4" size="2.54" layer="91" font="vector" ratio="15">thingSoC Reference Design
+Open Source Sockets for IoT</text>
 </plain>
 <instances>
