File: TSOC_RS485_EM/TSOC_RS485_EM.sch (EAGLE design)
At the start: 53 parts, among them Q1 FDC6420C, Q2 MOSFET-NCHANNELAO3404A, U1 ST1480ACSOIC, U2 ATMEGA328, U3 MIC5219 3.3V, U4 NCP361SNT1G, X1 8MHZ

Commit message: update to Rev6.0
Parts:
- removed D8, D9: (no value), PatternAgents-ProtoPads:WPAD-1-0402
- removed R17, R18, R19, R20, R21: DNP, TSOC-MODBUS-ESM:RESISTOR0402
- removed SJ3: JMP-2-NC, TSOC-MODBUS-ESM:JMP-2-NC
- added J10, J6, J7, J8, J9: (no value), TSOC_RS485_EM:JMP-2-NO
- added J11, J12, J13: JMP-2-NC, TSOC-MODBUS-ESM:JMP-2-NC
- added J3, J4, J5: JMP-3-1_2, TSOC_RS485_EM:JMP-3-1_2
- added JP1: (no value), TSOC_RS485_EM:M04PTH
- RS485: device SparkFun-Connectors:M04SCREW -> TSOC_RS485_EM:M04SCREW
- U$1: value TSOC-PCB-EM-BB -> TSOC-PCB-EM-45; device TSOC_RS485_EM:TSOC-PCB-EM-BB -> TSOC_RS485_EM:TSOC-PCB-EM-45
- renumbered LED_A2 to LED_G, LED_A3 to LED_R, LED_D4 to LED_B, LED_D5 to LED_Y, SJ1 to J2, SJ2 to J1
Connections:
- removed net A6: TSOC.!ATN, U2.ADC6
- removed net A7: TSOC.!IRQ, U2.ADC7
- new net DE: J4.2, R3.1, U1./RE, U1.DE
- new net DI: J5.2, U1.DI
- new net N$1: J13.1, TSOC.SS2
- new net TSOC_D8: J12.1, TSOC.IO1
- new net TSOC_D9: J11.1, TSOC.IO2
- net A0: now also TSOC.!IRQ; no longer TSOC.!DTR
- net AO: now also JP1.2
- net AREF: now also U2.ADC7
- net BO: now also JP1.4
- net D0: now also J10.2, J3.1; no longer R19.2, R20.2, SJ3.1
- net D1: now also J5.1, J9.2; no longer R18.2, R21.2, U1.DI
- net D2: now also J4.1, J6.2; no longer R17.2, R3.1, U1./RE, U1.DE
- net D4: now also TSOC.!DTR; no longer R2.2, TSOC.IO2
- net D5: now also J13.2, J4.3; no longer R1.2, TSOC.IO1
- net D6: now also TSOC.SS1; no longer TSOC.SS2
- net D7: now also TSOC.!ATN; no longer TSOC.SS1
- net D8: now also J12.2, J3.3, J8.2, R2.2; no longer D8.1
- net D9: now also J11.2, J5.3, J7.2, R1.2; no longer D9.1
- net EXT_5V0: now also JP1.1
- net GND: now also JP1.3
- net RXD: now also J3.2; no longer SJ3.2
- net TSOC_CTS: now also J6.1; no longer R17.1
- net TSOC_RXD: now also J10.1, J8.1; no longer R18.1, R19.1
- net TSOC_TXD: now also J7.1, J9.1; no longer R20.1, R21.1
- net VCC: now also U2.ADC6
Other:
- note added: "ThingSoC Serial Port Selection"
- note removed: "ThingSoC Base (or Expansion) Board Selection"
- moved on the sheet: R10, R6
