File: TSOC_RS485_EM/revisions/TSOC_RS485_EM_R4_0.brd (EAGLE design)
At the start: 43.2 x 25.4 mm, 54 parts, among them Q1 FDC6420C, Q2 MOSFET-NCHANNELAO3404A, U1 ST1480ACSOIC, U2 ATMEGA328, U3 MIC5219 3.3V, U4 NCP361SNT1G, X1 8MHZ

Commit message: update to revision 5.0
Parts:
- removed C10: 22uF, rcl:SMC_B
- removed D8, D9: (no value), PatternAgents-ProtoPads:WPAD-1-0402
- removed LED_D4, LED_D5: (no value), TSOC-MODBUS-ESM:LED-0603
- removed R16, R24: 1K, TSOC-MODBUS-ESM:0402-RES
- removed R17, R18, R19, R20, R21: DNP, TSOC-MODBUS-ESM:0402-RES
- removed R22, R23: 4K7, TSOC-MODBUS-ESM:0402-RES
- removed SJ3: JMP-2-NC, TSOC-MODBUS-ESM:JMP-2-NC
- added LED_D7, LED_D8: (no value), TSOC-MODBUS-ESM:LED-0603
- added RTERM: 120, TSOC-MODBUS-ESM:0402-RES
- C9: value 0.1uF -> 22uF; device TSOC-MODBUS-ESM:0402-CAP -> rcl:SMC_B
- R10: value DNP -> 1K
- R11: value 4K7 -> DNP
- R12, R8: value 10K -> 1K
- R13: value 100 -> 4K7
- R15: value 6K8 -> 1K
- R4: value 4K7 -> 10K
- R5: value 56 -> 100
- R6: value DNP -> 4K7
- R7: value 120 -> 6K8
- R9: value 56 -> DNP
- U$1: device TSOC_RS485_EM:TSOC-EM-BB -> TSOC-MODBUS-ESM:TSOC-EM-BB
- X1: value 8MHZ -> RESONATORSMD; device TSOC_RS485_EM:RESONATOR-SMD -> SparkFun:RESONATOR-SMD
- moved R8 33.5 mm to (5.08, 21.6), turned to 0 degrees
- moved R4 30.2 mm to (33.3, 15.5), turned to 90 degrees
- moved C7 25.3 mm to (11.2, 15.2), turned to 270 degrees
- moved R6 24.8 mm to (14.0, 18.8), turned to 90 degrees
- moved R13 24.1 mm to (29.2, 21.6), turned to 90 degrees
- moved C8 22.7 mm to (32.5, 19.3)
- moved R11 22.4 mm to (24.9, 21.6), turned to 270 degrees
- moved R9 20.7 mm to (22.4, 21.6), turned to 270 degrees
- moved R14 19.8 mm to (32.5, 21.6)
- moved R10 16.6 mm to (23.6, 21.6), turned to 270 degrees
- moved R12 15.8 mm to (26.2, 21.6), turned to 270 degrees
- moved R7 13.8 mm to (12.4, 20.1), turned to 90 degrees
- moved C5 12.5 mm to (31.8, 10.4)
- moved R5 10.9 mm to (6.86, 18.0), turned to 270 degrees
- moved R3 10.2 mm to (12.7, 15.2), turned to 90 degrees
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Connections:
- removed net !JDBG: R6.2, TSOC.1E
- removed net AO: R7.1, R9.1, RS485.2
- removed net BO: R5.1, R7.2, RS485.4
- removed net JTDO: R10.2, TSOC.2E
- removed net LEDB: LED_D4.C, R2.1
- removed net LEDG: LED_A2.C, R16.1
- removed net LEDR: LED_A3.C, R24.1
- removed net LEDY: LED_D5.C, R1.1
- removed net RXD: SJ3.2, U1.1
- removed net TSOC_CTS: R17.1, TSOC.6C
- removed net TSOC_RXD: R18.1, R19.1, TSOC.7C
- removed net TSOC_TXD: R20.1, R21.1, TSOC.8C
- new net LED_A2: LED_A2.C, R8.1
- new net N$2: LED_D7.C, R2.1
- new net N$3: LED_A3.C, R15.1
- new net N$4: LED_D8.C, R1.1
- new net TSOC_D0: R10.1, R9.1, TSOC.7C
- new net TSOC_D1: R11.1, R12.1, TSOC.8C
- net !5V0_FAULT: now also R3.1; no longer R12.1
- net !JRST: now also C4.1; no longer C7.1
- net !RST: now also C4.2, R4.1; no longer C7.2, R10.1, R8.1
- net 5V0: now also C7.1, C9.+, R3.2; no longer C10.+, C8.1, R12.2
- net A: now also RS485.4, RTERM.1, U1.7; no longer R11.2, R9.2, U1.6
- net A2: now also R8.2; no longer R16.2
- net A3: now also R15.2; no longer R24.2
- net A4: now also R14.2; no longer R23.2
- net A5: now also R13.2; no longer R22.2
- net AREF: now also C5.2; no longer C4.2
- net B: now also RS485.2, RTERM.2, U1.6; no longer R4.1, R5.2, U1.7
- net D0: now also R10.2, R11.2; no longer R19.2, R20.2, SJ3.1
- net D1: now also R12.2, R9.2; no longer R18.2, R21.2, U1.4
- net D2: now also TSOC.6C; no longer R17.2, R3.1, U1.2, U1.3
- net D4: now also U1.4; no longer R2.2, TSOC.1B
- net D5: now also U1.2, U1.3; no longer R1.2, TSOC.2B
- net D6: now also U1.1
- net D7: now also R2.2, TSOC.1B; no longer TSOC.4B
- net D8: now also R1.2, TSOC.2B; no longer D8.1
- net D9: now also TSOC.4B; no longer D9.1
- net EXT_5V0: now also R5.1; no longer R13.1
- net GND: now also C7.2, C9.-, R7.2; no longer C10.-, C4.1, C9.2, R15.2, R4.2
- net NGATE: now also R5.2, R6.1; no longer R13.2, R14.1
- net PGATE: now also R6.2, R7.1; no longer R14.2, R15.1
- net VCC: now also C8.1, LED_D7.A, LED_D8.A, R13.1, R14.1, R4.2; no longer C5.2, C9.1, LED_D4.A, LED_D5.A, R11.1, R22.1, R23.1, R3.2, R6.1, R8.2
Routing:
- net VCC: track 156.2 -> 107.6 mm, vias 15 -> 9
- net D2: track 32.1 -> 10.5 mm, vias 4 -> 0
- net D4: track 29.3 -> 11.2 mm, vias 1 -> 2
- net GND: track 159.4 -> 144.5 mm, vias 14 -> 12
- net RXD: track 13.8 -> 0.00 mm
- net D1: track 50.7 -> 37.5 mm, vias 5 -> 4
- net D5: track 25.0 -> 12.2 mm
- net D8: track 10.7 -> 22.6 mm, vias 1 -> 0
- net D7: track 13.1 -> 22.5 mm, vias 0 -> 1
- net AO: track 8.92 -> 0.00 mm
- net D0: track 33.8 -> 26.7 mm, vias 3 -> 2
- net B: track 4.69 -> 10.9 mm, vias 0 -> 1
- net !JDBG: track 6.08 -> 0.00 mm
- net BO: track 5.80 -> 0.00 mm
- net JTDO: track 5.59 -> 0.00 mm
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Other:
- board size 43.2 x 25.4 mm -> 40.6 x 25.4 mm
- board text added: "!ATN"
- board text added: "!CS"
- board text added: "!CTS"
- board text added: "!DCD"
- board text added: "!DSR"
- board text added: "!DTR/RST"
- board text added: "!RI"
- board text added: "!RTS"
- board text added: "5VDC"
- board text added: "CTS"
- board text added: "IO1"
- board text added: "IO2"
- board text added: "MISO"
- board text added: "MOSI"
- board text added: "NC"
- board text added: "RXD"
- board text added: "Rev 4.0 (AVR Version)"
- board text added: "SCK"
- board text added: "SCL"
- board text added: "SDA"
- board text added: "SS1"
- board text added: "SS2"
- board text added: "TXD"
- board text removed: "!DBG"
- board text removed: "!RST"
- board text removed: "5VDC_IN"
- board text removed: "A1"
- board text removed: "A2"
- board text removed: "A3"
- board text removed: "A4"
- board text removed: "A5"
- board text removed: "A6"
- board text removed: "A7"
- board text removed: "D0"
- board text removed: "D1"
- board text removed: "D10"
- board text removed: "D11"
- board text removed: "D12"
- board text removed: "D13"
- board text removed: "D2"
- board text removed: "D3"
- board text removed: "D4"
- board text removed: "D5"
- board text removed: "D6"
- board text removed: "D7"
- board text removed: "RS-485"
- board text removed: "Rev 5.0 (AVR Version)"
