File: TSOC_RS485_EM/revisions/TSOC_RS485_EM_R4_0.sch (EAGLE design)
At the start: 53 parts, among them Q1 FDC6420C, Q2 MOSFET-NCHANNELAO3404A, U1 ST1480ACSOIC, U2 ATMEGA328, U3 MIC5219 3.3V, U4 NCP361SNT1G, X1 8MHZ

Commit message: update to revision 5.0
Parts:
- removed C10: 22uF, rcl:CPOL-EUSMCB
- removed D8, D9: (no value), PatternAgents-ProtoPads:WPAD-1-0402
- removed R16, R24: 1K, TSOC-MODBUS-ESM:RESISTOR0402
- removed R17, R18, R19, R20, R21: DNP, TSOC-MODBUS-ESM:RESISTOR0402
- removed R22, R23: 4K7, TSOC-MODBUS-ESM:RESISTOR0402
- removed SJ3: JMP-2-NC, TSOC-MODBUS-ESM:JMP-2-NC
- added RTERM: 120, TSOC-MODBUS-ESM:RESISTOR0402
- C9: value 0.1uF -> 22uF; device TSOC-MODBUS-ESM:CAP0402-CAP -> rcl:CPOL-EUSMCB
- R10: value DNP -> 1K
- R11: value 4K7 -> DNP
- R12, R8: value 10K -> 1K
- R13: value 100 -> 4K7
- R15: value 6K8 -> 1K
- R4: value 4K7 -> 10K
- R5: value 56 -> 100
- R6: value DNP -> 4K7
- R7: value 120 -> 6K8
- R9: value 56 -> DNP
- U$1: device TSOC_RS485_EM:TSOC-PCB-EM-BB -> TSOC-MODBUS-ESM:TSOC-PCB-EM-BB
- X1: value 8MHZ -> RESONATORSMD; device TSOC_RS485_EM:RESONATOR8MHZ -> SparkFun:RESONATORSMD
- renumbered LED_D4 to LED_D7, LED_D5 to LED_D8
Connections:
- net LEDB renamed N$2
- net LEDY renamed N$4
- removed net !JDBG: R6.2, TSOC.!JDBG
- removed net AO: R7.1, R9.1, RS485.2
- removed net BO: R5.1, R7.2, RS485.4
- removed net JTDO: R10.2, TSOC.JTDO
- removed net LEDG: LED_A2.C, R16.1
- removed net LEDR: LED_A3.C, R24.1
- removed net RXD: SJ3.2, U1.RO
- removed net TSOC_CTS: R17.1, TSOC.!CTS
- removed net TSOC_RXD: R18.1, R19.1, TSOC.RXD
- removed net TSOC_TXD: R20.1, R21.1, TSOC.TXD
- new net LED_A2: LED_A2.C, R8.1
- new net N$3: LED_A3.C, R15.1
- new net TSOC_D0: R10.1, R9.1, TSOC.RXD
- new net TSOC_D1: R11.1, R12.1, TSOC.TXD
- net !5V0_FAULT: now also R3.1; no longer R12.1
- net !JRST: now also C4.1; no longer C7.1
- net !RST: now also C4.2, R4.1; no longer C7.2, R10.1, R8.1
- net 5V0: now also C7.1, C9.+, R3.2; no longer C10.+, C8.1, R12.2
- net A: now also RS485.4, RTERM.1, U1.B; no longer R11.2, R9.2, U1.A
- net A2: now also R8.2; no longer R16.2
- net A3: now also R15.2; no longer R24.2
- net A4: now also R14.2; no longer R23.2
- net A5: now also R13.2; no longer R22.2
- net AREF: now also C5.2; no longer C4.2
- net B: now also RS485.2, RTERM.2, U1.A; no longer R4.1, R5.2, U1.B
- net D0: now also R10.2, R11.2; no longer R19.2, R20.2, SJ3.1
- net D1: now also R12.2, R9.2; no longer R18.2, R21.2, U1.DI
- net D2: now also TSOC.!CTS; no longer R17.2, R3.1, U1./RE, U1.DE
- net D4: now also U1.DI; no longer R2.2, TSOC.IO2
- net D5: now also U1./RE, U1.DE; no longer R1.2, TSOC.IO1
- net D6: now also U1.RO
- net D7: now also R2.2, TSOC.IO2; no longer TSOC.SS1
- net D8: now also R1.2, TSOC.IO1; no longer D8.1
- net D9: now also TSOC.SS1; no longer D9.1
- net EXT_5V0: now also R5.1; no longer R13.1
- net GND: now also C7.2, C9.-, R7.2; no longer C10.-, C4.1, C9.2, R15.2, R4.2
- net NGATE: now also R5.2, R6.1; no longer R13.2, R14.1
- net PGATE: now also R6.2, R7.1; no longer R14.2, R15.1
- net VCC: now also C8.1, R13.1, R14.1, R4.2; no longer C5.2, C9.1, R11.1, R22.1, R23.1, R3.2, R6.1, R8.2
Other:
- moved on the sheet: C1, C2, C4, C5, C6, C7, C8, Q1N-CH, Q1P-CH, Q2, R10, R11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
