File: TSOC_RS485_EM/revisions/TSOC_RS485_EM_R5_1.brd (EAGLE design)
At the start: 43.2 x 25.4 mm, 54 parts, among them Q1 FDC6420C, Q2 MOSFET-NCHANNELAO3404A, U1 ST1480ACSOIC, U2 ATMEGA328, U3 MIC5219 3.3V, U4 NCP361SNT1G, X1 8MHZ

Commit message: update to revision 5.0
Parts:
- moved C5 2.54 mm to (21.8, 11.2)
- moved R21 2.54 mm to (28.7, 21.6)
- moved D9 2.54 mm to (17.8, 5.33)
- moved Q1 2.54 mm to (11.2, 18.5)
- moved R12 2.54 mm to (14.2, 15.2)
- moved R15 2.54 mm to (14.0, 20.1)
- moved U3 2.54 mm to (17.0, 14.5)
- moved U4 2.54 mm to (9.91, 14.7)
- moved LED_A2 2.54 mm to (1.78, 21.6)
- moved LED_A3 2.54 mm to (1.78, 23.4)
- moved LED_D4 2.54 mm to (1.78, 3.56)
- moved LED_D5 2.54 mm to (1.78, 1.78)
- moved R11 2.54 mm to (7.11, 12.2)
- moved R13 2.54 mm to (7.87, 18.0)
- moved R16 2.54 mm to (5.08, 21.6)
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Other:
- board text added: "!DBG"
- board text added: "!RST"
- board text added: "5VDC_IN"
- board text added: "A1"
- board text added: "A2"
- board text added: "A3"
- board text added: "A4"
- board text added: "A5"
- board text added: "A6"
- board text added: "A7"
- board text added: "D0"
- board text added: "D1"
- board text added: "D10"
- board text added: "D11"
- board text added: "D12"
- board text added: "D13"
- board text added: "D2"
- board text added: "D3"
- board text added: "D4"
- board text added: "D5"
- board text added: "D6"
- board text added: "D7"
- board text added: "RS-485"
- board text removed: "!ATN"
- board text removed: "!CS"
- board text removed: "!CTS"
- board text removed: "!DCD"
- board text removed: "!DSR"
- board text removed: "!DTR/RST"
- board text removed: "!RI"
- board text removed: "!RTS"
- board text removed: "5VDC"
- board text removed: "CTS"
- board text removed: "IO1"
- board text removed: "IO2"
- board text removed: "MISO"
- board text removed: "MOSI"
- board text removed: "NC"
- board text removed: "RXD"
- board text removed: "SCK"
- board text removed: "SCL"
- board text removed: "SDA"
- board text removed: "SS1"
- board text removed: "SS2"
- board text removed: "TXD"
