File: TSOC_RS485_EM/revisions/rev7_1/TSOC_RS485_EM.sch (EAGLE design)
At the start: 62 parts, among them J1 JMP-3-1_2, J11 JMP-2-NC, J12 JMP-2-NC, J13 JMP-2-NC, J2 JMP-2-NC, J3 JMP-3-1_2, J4 JMP-3-1_2, J5 JMP-3-1_2, Q1 FDC6420C, Q2 MOSFET-NCHANNELAO3404A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

Commit message: add product images
Other:
- note removed: "!JTAG"
- note removed: "!JTRST"
- note removed: "!RST"
- note removed: "JTCK"
- note removed: "JTDI"
- note removed: "JTDO"
- note removed: "JTMS"
- note removed: "MISO"
- note removed: "MOSI"
- note removed: "SCK"
- note removed: "SPI"
- note removed: "SSEL"
- note removed: "SWDCLK"
- note removed: "SWDIO"
Changed lines of the file:
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@@
 <text x="477.52" y="25.4" size="2.54" layer="91" font="vector" ratio="15">thingSoC Reference Design
 Open Source Sockets for IoT</text>
+<text x="104.14" y="182.88" size="1.6764" layer="91" font="vector" ratio="10" rot="MR0" align="center">POWER</text>
+<text x="104.14" y="177.8" size="1.6764" layer="91" font="vector" ratio="10" rot="MR0" align="center">GROUND</text>
 <text x="170.18" y="195.58" size="1.6764" layer="91" font="vector" ratio="10" rot="MR0" align="center">!DEBUG</text>
 <text x="170.18" y="193.04" size="1.6764" layer="91" font="vector" ratio="10" rot="MR0" align="center">!RTS</text>
@@
 <text x="170.18" y="182.88" size="1.6764" layer="91" font="vector" ratio="10" rot="MR0" align="center">POWER</text>
 <text x="170.18" y="177.8" size="1.6764" layer="91" font="vector" ratio="10" rot="MR0" align="center">GROUND</text>
-<text x="106.68" y="180.34" size="1.6764" layer="91" font="vector" ratio="10" rot="MR0" align="center">JTDI</text>
-<text x="106.68" y="193.04" size="1.6764" layer="91" font="vector" ratio="10" rot="MR0" align="center">JTDO</text>
-<text x="106.68" y="190.5" size="1.6764" layer="91" font="vector" ratio="10" rot="MR0" align="center">!JTRST</text>
-<text x="106.68" y="187.96" size="1.6764" layer="91" font="vector" ratio="10" rot="MR0" align="center">JTCK</text>
-<text x="106.68" y="185.42" size="1.6764" layer="91" font="vector" ratio="10" rot="MR0" align="center">JTMS</text>
-<text x="106.68" y="182.88" size="1.6764" layer="91" font="vector" ratio="10" rot="MR0" align="center">POWER</text>
-<text x="106.68" y="177.8" size="1.6764" layer="91" font="vector" ratio="10" rot="MR0" align="center">GROUND</text>
-<text x="106.68" y="195.58" size="1.6764" layer="91" font="vector" ratio="10" rot="MR0" align="center">!JTAG</text>
-<text x="96.52" y="187.96" size="1.6764" layer="91" font="vector" ratio="10" rot="MR0" align="center">SWDCLK</text>
-<text x="96.52" y="185.42" size="1.6764" layer="91" font="vector" ratio="10" rot="MR0" align="center">SWDIO</text>
-<text x="96.52" y="195.58" size="1.6764" layer="91" font="vector" ratio="10" rot="MR0" align="center">!JTAG</text>
-<text x="96.52" y="193.04" size="1.6764" layer="91" font="vector" ratio="10" rot="MR0" align="center">JTDO</text>
-<text x="96.52" y="190.5" size="1.6764" layer="91" font="vector" ratio="10" rot="MR0" align="center">!JTRST</text>
-<text x="96.52" y="182.88" size="1.6764" layer="91" font="vector" ratio="10" rot="MR0" align="center">POWER</text>
-<text x="96.52" y="180.34" size="1.6764" layer="91" font="vector" ratio="10" rot="MR0" align="center">JTDI</text>
-<text x="96.52" y="177.8" size="1.6764" layer="91" font="vector" ratio="10" rot="MR0" align="center">GROUND</text>
-<text x="86.36" y="187.96" size="1.6764" layer="91" font="vector" ratio="10" rot="MR0" align="center">SCK</text>
-<text x="86.36" y="185.42" size="1.6764" layer="91" font="vector" ratio="10" rot="MR0" align="center">SSEL</text>
-<text x="86.36" y="195.58" size="1.6764" layer="91" font="vector" ratio="10" rot="MR0" align="center">SPI</text>
-<text x="86.36" y="193.04" size="1.6764" layer="91" font="vector" ratio="10" rot="MR0" align="center">MOSI</text>
-<text x="86.36" y="190.5" size="1.6764" layer="91" font="vector" ratio="10" rot="MR0" align="center">!RST</text>
-<text x="86.36" y="182.88" size="1.6764" layer="91" font="vector" ratio="10" rot="MR0" align="center">POWER</text>
-<text x="86.36" y="180.34" size="1.6764" layer="91" font="vector" ratio="10" rot="MR0" align="center">MISO</text>
-<text x="86.36" y="177.8" size="1.6764" layer="91" font="vector" ratio="10" rot="MR0" align="center">GROUND</text>
 </plain>
 <instances>
