File: TSOC_RS485_EM/revisions/rev8_0/TSOC_RS485_EM.brd (EAGLE design)
At the start: 53.3 x 30.5 mm, 65 parts, among them J1 JMP-3-1_2, J11 JMP-2-NC, J12 JMP-2-NC, J13 JMP-2-NC, J2 JMP-2-NC, J3 JMP-3-1_2, J4 JMP-3-1_2, J5 JMP-3-1_2, Q1 FDC6420C, Q2 MOSFET-NCHANNELAO3404A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

Commit message: add product images
Parts:
- removed R10, R6: DNP, PatternAgents-ProtoPads:EIA-0402-MIN
Connections:
- new net !JTAG: J14.1
- net !JDBG: no longer R6.2, TSOC.1E
- net !RST: no longer R10.1
- net D10: now also J14.9
- net D11: now also J14.3
- net D12: now also J14.13
- net D13: now also J14.7
- net JTDO: no longer R10.2, TSOC.2E
- net VCC: no longer R6.1
Routing:
- net D12: track 4.09 -> 41.9 mm
- net D10: track 6.43 -> 44.2 mm
- net D13: track 8.29 -> 37.9 mm
- net D11: track 11.3 -> 30.5 mm
- net JTDO: track 8.91 -> 0.00 mm
- net !JDBG: track 8.53 -> 0.00 mm
- net GND: track 152.4 -> 153.3 mm
- net VCC: track 144.8 -> 144.3 mm
Other:
- board text added: "Rev 8.0 (AVR Version)"
- board text removed: "Rev 7.1 (AVR Version)"
