File: TSOC_RS485_EM/revisions/rev8_0/TSOC_RS485_EM.sch (EAGLE design)
At the start: 62 parts, among them J1 JMP-3-1_2, J11 JMP-2-NC, J12 JMP-2-NC, J13 JMP-2-NC, J2 JMP-2-NC, J3 JMP-3-1_2, J4 JMP-3-1_2, J5 JMP-3-1_2, Q1 FDC6420C, Q2 MOSFET-NCHANNELAO3404A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

Commit message: add product images
Parts:
- removed R10, R6: DNP, PatternAgents-ProtoPads:RESISTOR0402-MIN
Connections:
- new net !JTAG: J14.1
- net !JDBG: no longer R6.2, TSOC.!JDBG
- net !RST: no longer R10.1
- net D10: now also J14.9
- net D11: now also J14.3
- net D12: now also J14.13
- net D13: now also J14.7
- net JTDO: no longer R10.2, TSOC.JTDO
- net VCC: no longer R6.1
Changed lines of the file:
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@@
 <part name="C9" library="PatternAgents-ProtoPads" deviceset="CAP" device="TYP" value="0.1uF"/>
 <part name="GND3" library="supply1" deviceset="GND" device=""/>
-<part name="R10" library="PatternAgents-ProtoPads" deviceset="RESISTOR" device="0402-MIN" value="DNP"/>
 <part name="GND4" library="supply1" deviceset="GND" device=""/>
 <part name="R9" library="PatternAgents-ProtoPads" deviceset="RESISTOR" device="0402-MIN" value="56"/>
@@
 <part name="GND5" library="supply1" deviceset="GND" device=""/>
 <part name="R7" library="PatternAgents-ProtoPads" deviceset="RESISTOR" device="0402-MIN" value="120"/>
-<part name="R6" library="PatternAgents-ProtoPads" deviceset="RESISTOR" device="0402-MIN" value="DNP"/>
 <part name="R3" library="PatternAgents-ProtoPads" deviceset="RESISTOR" device="0402-MIN" value="10K"/>
 <part name="C5" library="PatternAgents-ProtoPads" deviceset="CAP" device="TYP" value="0.1uF"/>
@@
 <instance part="C9" gate="G$1" x="520.7" y="307.34"/>
 <instance part="GND3" gate="1" x="520.7" y="297.18"/>
-<instance part="R10" gate="R" x="198.12" y="106.68" rot="R180"/>
 <instance part="GND4" gate="1" x="469.9" y="83.82"/>
 <instance part="R9" gate="R" x="441.96" y="114.3" rot="R180"/>
@@
 <instance part="GND5" gate="1" x="431.8" y="78.74"/>
 <instance part="R7" gate="R" x="457.2" y="106.68" rot="R270"/>
-<instance part="R6" gate="R" x="198.12" y="99.06" rot="R180"/>
 <instance part="R3" gate="R" x="368.3" y="121.92" rot="R90"/>
 <instance part="C5" gate="G$1" x="88.9" y="375.92" smashed="yes" rot="R90">
@@
 </segment>
 <segment>
-<pinref part="R10" gate="R" pin="1"/>
-<wire x1="203.2" y1="106.68" x2="208.28" y2="106.68" width="0.1524" layer="91"/>
-<label x="208.28" y="106.68" size="1.27" layer="95" font="vector" ratio="10" xref="yes"/>
-</segment>
-<segment>
 <pinref part="J14" gate="G$1" pin="5"/>
 <wire x1="129.54" y1="190.5" x2="119.38" y2="190.5" width="0.1524" layer="91"/>
@@
 <label x="182.88" y="88.9" size="1.27" layer="95" font="vector" ratio="10" xref="yes"/>
 </segment>
+<segment>
+<pinref part="J14" gate="G$1" pin="7"/>
+<wire x1="129.54" y1="187.96" x2="119.38" y2="187.96" width="0.1524" layer="91"/>
+<label x="119.38" y="187.96" size="1.27" layer="95" font="vector" ratio="10" rot="R180" xref="yes"/>
+</segment>
 </net>
 <net name="D12" class="0">
@@
 <label x="182.88" y="86.36" size="1.27" layer="95" font="vector" ratio="10" xref="yes"/>
 </segment>
+<segment>
+<pinref part="J14" gate="G$1" pin="13"/>
+<wire x1="129.54" y1="180.34" x2="119.38" y2="180.34" width="0.1524" layer="91"/>
+<label x="119.38" y="180.34" size="1.27" layer="95" font="vector" ratio="10" rot="R180" xref="yes"/>
+</segment>
 </net>
 <net name="D11" class="0">
@@
 <label x="182.88" y="83.82" size="1.27" layer="95" font="vector" ratio="10" xref="yes"/>
 </segment>
+<segment>
+<pinref part="J14" gate="G$1" pin="3"/>
+<wire x1="129.54" y1="193.04" x2="119.38" y2="193.04" width="0.1524" layer="91"/>
+<label x="119.38" y="193.04" size="1.27" layer="95" font="vector" ratio="10" rot="R180" xref="yes"/>
+</segment>
 </net>
 <net name="XOUT" class="0">
@@
 <wire x1="165.1" y1="81.28" x2="182.88" y2="81.28" width="0.1524" layer="91"/>
 <label x="182.88" y="81.28" size="1.27" layer="95" font="vector" ratio="10" xref="yes"/>
+</segment>
+<segment>
+<pinref part="J14" gate="G$1" pin="9"/>
+<wire x1="129.54" y1="185.42" x2="119.38" y2="185.42" width="0.1524" layer="91"/>
+<label x="119.38" y="185.42" size="1.27" layer="95" font="vector" ratio="10" rot="R180" xref="yes"/>
 </segment>
 </net>
@@
 <wire x1="147.32" y1="279.4" x2="152.4" y2="279.4" width="0.1524" layer="91"/>
 <label x="152.4" y="279.4" size="1.27" layer="95" font="vector" ratio="10" xref="yes"/>
-</segment>
-<segment>
-<pinref part="R6" gate="R" pin="1"/>
-<wire x1="203.2" y1="99.06" x2="208.28" y2="99.06" width="0.1524" layer="91"/>
-<label x="208.28" y="99.06" size="1.27" layer="95" font="vector" ratio="10" xref="yes"/>
 </segment>
 <segment>
@@
 <net name="JTDO" class="0">
 <segment>
-<pinref part="TSOC" gate="TSOC" pin="JTDO"/>
-<pinref part="R10" gate="R" pin="2"/>
-<wire x1="165.1" y1="106.68" x2="193.04" y2="106.68" width="0.1524" layer="91"/>
-</segment>
-<segment>
 <pinref part="J14" gate="G$1" pin="4"/>
 <wire x1="144.78" y1="193.04" x2="154.94" y2="193.04" width="0.1524" layer="91"/>
@@
 </net>
 <net name="!JDBG" class="0">
-<segment>
-<pinref part="TSOC" gate="TSOC" pin="!JDBG"/>
-<wire x1="165.1" y1="104.14" x2="190.5" y2="104.14" width="0.1524" layer="91"/>
-<wire x1="190.5" y1="104.14" x2="190.5" y2="99.06" width="0.1524" layer="91"/>
-<pinref part="R6" gate="R" pin="2"/>
-<wire x1="190.5" y1="99.06" x2="193.04" y2="99.06" width="0.1524" layer="91"/>
-</segment>
 <segment>
 <wire x1="144.78" y1="195.58" x2="154.94" y2="195.58" width="0.1524" layer="91"/>
@@
 </segment>
 </net>
+<net name="!JTAG" class="0">
+<segment>
+<pinref part="J14" gate="G$1" pin="1"/>
+<wire x1="129.54" y1="195.58" x2="119.38" y2="195.58" width="0.1524" layer="91"/>
+<label x="119.38" y="195.58" size="1.27" layer="95" font="vector" ratio="10" rot="R180" xref="yes"/>
+</segment>
+</net>
